File: MasterBoard.sch (EAGLE design)
At the start: 44 parts, among them IC1 MAX6954AAX+, IC2 MCP23017SO, U6 MAX3232

Commit message: Added renders, readme, cleanup
Parts:
- removed A0, A1, A2: (no value), jumper:SJ
- removed C13: 1.0uF, SparkFun-Capacitors:1.0UF-0805-25V-10%
- removed C22, C23, C24: 0.1uF, SparkFun-Capacitors:1.0UF-0805-25V-10%
- removed DE9FEMALE: EDGEMOUNTDE9, Serial:EDGEMOUNTDE9
- removed IC2: MCP23017SO, adafruit:MCP23017SO
- removed J1: (no value), SparkFun-Connectors:CONN_09
- removed JP1: (no value), microbuilder:HEADER-1X16ROUND
- removed JP3: (no value), microbuilder:HEADER-1X12
- removed R1, R10, R11, R12, R13, R14, R15, R16, R17, R2, R3, R4, R5, R6, R7, R8, R9: 10k, resistor:R-US_M0805
- removed R18: 56k, resistor:R-US_M0805
- removed U$1: HDSP-A27C, Segment displays:HDSP-A27C
- removed U$10, U$7, U$8, U$9: KEYSTONESTANDOFF, Segment displays:KEYSTONESTANDOFF
- removed U$2, U$3, U$6: RM107772BCB, Segment displays:RM107772BCB
- removed U$5: OS102011MA1QN1, FPC:OS102011MA1QN1
- removed U6: MAX3232, SparkFun-IC-Comms:MAX2323SOIC16
- added A10, A11, A9: (no value), microbuilder:SOLDERJUMPERREFLOW_NOPASTE
- added A6, A7, A8: (no value), jumper:SJ
- added C4: 1.0uF, SparkFun-Capacitors:1.0UF-0805-25V-10%
- added D19, D20, D21, D22, D23, D24, D25, D26, D27, D28, D29, D30, D31, D32, D33, D34, D35, D36: 200mA/100V/1V, SparkFun-DiscreteSemi:DIODE-1N4148
- added D2: 1N4148, adafruit:DIODESOD-323F
- added DE9FEMALE1: EDGEMOUNTDE9, Serial:EDGEMOUNTDE9
- added HT16K1: (no value), microbuilder:HT16K33_SOP28_SKINNY
- added JP2: (no value), microbuilder:HEADER-1X16ROUND
- added JP4: (no value), microbuilder:HEADER-1X12
- added R35, R36, R37, R38, R39: 10k, resistor:R-US_M0805
- added R40, R41: 10K, microbuilder:RESISTOR0805_NOOUTLINE
- added R42, R43, R44: 47K, microbuilder:RESISTOR0805_NOOUTLINE
- added S_10, S_11, S_12, S_13, S_14, S_15, S_16, S_17, S_18, S_19, S_A1, S_B1, S_BACK1, S_C1, S_D1, S_E1, S_ENTER1, S_F1: MX, SparkFun-Switches:MOMENTARY-SWITCH-SPST-LED-PTH-CHERRY
- added U$11: BIG14SEG, Segment displays:BIG14SEG
- added U$12, U$17, U$18: RM107772BCB, Segment displays:RM107772BCB
- added U$15: OS102011MA1QN1, FPC:OS102011MA1QN1
- added U1: MAX3232, SparkFun-IC-Comms:MAX2323SOIC16
- C1: value 22pf -> 0.1uF; device SparkFun-Capacitors:1.0UF-0805-25V-(+80/-20%) -> SparkFun-Capacitors:1.0UF-0805-25V-10%
- C2: value 100nF -> 0.1uF; device SparkFun-Capacitors:1.0UF-0805-25V-(+80/-20%) -> SparkFun-Capacitors:1.0UF-0805-25V-10%
- C3: value 47uF -> 0.1uF; device adafruit:C-USC1206 -> SparkFun-Capacitors:1.0UF-0805-25V-10%
- IC1: value MAX6954AAX+ -> MCP23017SO; device SamacSys_Parts:MAX6954AAX+ -> adafruit:MCP23017SO
Connections:
- removed net +3V3: A0.2, A1.2, A2.2, C2.2, C3.2, IC1.V+_1, IC1.V+_2, IC2.!RESET, IC2.VDD, JP1.15, R16.2, R17.2, U$2.C, U$3.C, U$6.C
- removed net 3V3: U6.VCC
- removed net N$10: IC1.O12, U$1.P
- removed net N$11: IC1.O13, U$1.G
- removed net N$12: IC1.O14, U$1.H
- removed net N$13: IC1.O15, U$1.K
- removed net N$14: IC1.O16, U$1.L
- removed net N$15: IC1.O17, U$1.M
- removed net N$16: IC1.O18, U$1.DP
- removed net N$17: IC1.O1, U$1.COM2
- removed net N$18: C22.2, U6.C1-
- removed net N$19: C22.1, U6.C1+
- removed net N$20: C23.1, U6.C2+
- removed net N$21: C23.2, U6.C2-
- removed net N$22: C24.1, U6.V+
- removed net N$5: IC1.O6, U$1.D
- removed net N$6: IC1.O8, U$1.E
- removed net N$7: IC1.O9, U$1.F
- removed net N$8: IC1.O10, U$1.N
- removed net N$9: IC1.O11, U$1.J
- new net A0: A10.2, HT16K1.ROW2/A0, U$11.C
- new net A1: A9.2, HT16K1.ROW1/A1, U$11.B
- new net A2: A11.2, HT16K1.ROW0/A2, U$11.A
- new net COM0: D2.A, HT16K1.COM0/AD, U$11.COM1
- new net COM1: HT16K1.COM1/KS0, U$11.COM2
- new net N$32: D23.A, S_ENTER1.1
- new net N$33: D22.A, S_F1.1
- new net N$34: D21.A, S_E1.1
- new net N$35: D20.A, S_D1.1
- new net N$36: D19.A, S_C1.1
- new net N$50: C1.2, U1.C1-
- new net N$51: C1.1, U1.C1+
- new net N$52: C2.1, U1.C2+
- new net N$53: C2.2, U1.C2-
- new net N$54: C3.1, U1.V+
- new net N$55: C4.1, U1.V-
- new net N$56: DE9FEMALE1.P2, DE9FEMALE1.P5, DE9FEMALE1.P9
- new net N$57: A6.1, IC1.A0, R35.2
- new net N$58: A7.1, IC1.A1, R36.2
- new net N$59: A8.1, IC1.A2, R37.2
- new net N$60: IC1.INTB, R38.1
- new net N$61: IC1.INTA, R39.1
- new net N$62: A9.1, R42.2
- new net N$63: A10.1, R43.2
- new net N$64: HT16K1.ROW3/K1, U$11.D
- new net N$65: HT16K1.ROW4/K2, U$11.E
- new net N$66: HT16K1.ROW5/K3, U$11.F
- new net N$67: HT16K1.ROW6/K4, U$11.N
- new net N$68: HT16K1.ROW7/K5, U$11.J
- new net N$69: D2.C, R42.1, R43.1, R44.1
- new net N$70: A11.1, R44.2
- new net N$71: HT16K1.ROW8/K6, U$11.P
- new net N$72: HT16K1.ROW9/K7, U$11.G
- new net N$73: HT16K1.ROW10/K8, U$11.H
- new net N$74: HT16K1.ROW11/K9, U$11.M
- new net N$75: HT16K1.ROW12/K10, U$11.L
- new net N$76: HT16K1.ROW13/K11, U$11.K
- new net N$77: HT16K1.ROW14/K12, U$11.DP
- new net VCC: A6.2, A7.2, A8.2, HT16K1.VDD, IC1.!RESET, IC1.VDD, JP2.15, R38.2, R39.2, R40.1, R41.1, U1.VCC
- net !RESET: now also JP2.16; no longer JP1.16
- net /CS: now also JP4.10; no longer IC1.!CS, JP3.10
- net A5: now also JP2.7; no longer JP1.7
- net AREF: now also JP2.14; no longer JP1.14
- net D13: now also JP4.4; no longer JP3.4
- net D9: now also JP4.8; no longer JP3.8
- net EN: now also JP4.2, U$15.P$2; no longer JP3.2, U$5.P$2
- net GND: now also C3.2, C4.2, DE9FEMALE1.P1, DE9FEMALE1.SHIELD, HT16K1.VSS, IC1.VSS, JP2.1, JP2.13, R35.1, R36.1, R37.1, U$12.C, U$15.P$1, U$17.C, U$18.C, U1.GND; no longer C1.2, C13.2, C2.1, C24.2, C3.1, DE9FEMALE.P1, DE9FEMALE.SHIELD, IC1.GND_1, IC1.GND_2, IC2.VSS, JP1.1, JP1.13, R1.1, R10.1, R11.1, R12.1, R13.1, R14.1, R15.1, R18.1, R2.1, R3.1, R4.1, R5.1, R6.1, R7.1, R8.1, R9.1, U$5.P$1, U6.GND
- net KC1: now also D19.C, D24.C, D29.C, D33.C, JP2.8; no longer J1.5, JP1.8
- net KC2: now also D20.C, D25.C, D30.C, D34.C, JP2.9; no longer J1.4, JP1.9
- net KC3: now also D21.C, D26.C, D31.C, D35.C, JP2.10; no longer J1.3, JP1.10
- net KC4: now also D22.C, D27.C, D32.C, D36.C, JP2.11; no longer J1.2, JP1.11
- net KC5: now also D23.C, D28.C, JP2.12; no longer J1.1, JP1.12
- net KR1: now also JP4.9, S_C1.2, S_D1.2, S_E1.2, S_ENTER1.2, S_F1.2; no longer J1.9, JP3.9
- net KR2: now also JP4.7, S_10.2, S_18.2, S_A1.2, S_B1.2, S_BACK1.2; no longer J1.8, JP3.7
- net KR3: now also JP4.6, S_13.2, S_14.2, S_16.2, S_17.2; no longer J1.7, JP3.6
- net KR4: now also JP4.5, S_11.2, S_12.2, S_15.2, S_19.2; no longer J1.6, JP3.5
- net MISO: now also JP2.4; no longer IC1.DIN, JP1.4
- net MOSI: now also JP2.5; no longer IC1.DOUT, JP1.5
- net N$1: now also D33.A, S_11.1; no longer IC1.O0, U$1.COM1
- net N$2: now also D34.A, S_19.1; no longer IC1.O2, U$1.A
- net N$23: now also D29.A, S_14.1; no longer C13.1, U6.V-
- net N$24: now also D30.A, S_17.1; no longer DE9FEMALE.P2, DE9FEMALE.P5, DE9FEMALE.P9
- net N$25: now also D31.A, S_16.1; no longer A0.1, IC2.A0, R13.2
- net N$26: now also D32.A, S_13.1; no longer A1.1, IC2.A1, R14.2
- net N$27: now also D24.A, S_10.1; no longer A2.1, IC2.A2, R15.2
- net N$28: now also D25.A, S_18.1; no longer IC2.INTB, R16.1
- net N$29: now also D26.A, S_A1.1; no longer IC2.INTA, R17.1
- net N$3: now also D35.A, S_15.1; no longer IC1.O4, U$1.B
- net N$30: now also D27.A, S_B1.1; no longer C1.1, IC1.OSC
- net N$31: now also D28.A, S_BACK1.1; no longer IC1.ISET, R18.2
- net N$4: now also D36.A, S_12.1; no longer IC1.O5, U$1.C
- net RM102-1: now also IC1.GPB6, U$18.1; no longer IC2.GPB6, R11.2, U$6.1
- net RM102-2: now also IC1.GPB7, U$18.2; no longer IC2.GPB7, R12.2, U$6.2
- net RM103-1: now also IC1.GPB0, U$17.1; no longer IC2.GPB0, R8.2, U$3.1
- net RM103-2: now also IC1.GPB1, U$17.2; no longer IC2.GPB1, R9.2, U$3.2
- net RM103-3: now also IC1.GPB2, U$17.3; no longer IC2.GPB2, R10.2, U$3.3
- net RM107-1: now also IC1.GPA1, U$12.1; no longer IC2.GPA1, R1.2, U$2.1
- net RM107-2: now also IC1.GPA2, U$12.2; no longer IC2.GPA2, R2.2, U$2.2
- net RM107-3: now also IC1.GPA3, U$12.3; no longer IC2.GPA3, R3.2, U$2.3
- net RM107-4: now also IC1.GPA4, U$12.4; no longer IC2.GPA4, R4.2, U$2.4
- net RM107-5: now also IC1.GPA5, U$12.5; no longer IC2.GPA5, R5.2, U$2.5
- net RM107-6: now also IC1.GPA6, U$12.6; no longer IC2.GPA6, R6.2, U$2.6
- net RM107-7: now also IC1.GPA7, U$12.7; no longer IC2.GPA7, R7.2, U$2.7
- net RXD: now also DE9FEMALE1.P3, U1.R1IN; no longer DE9FEMALE.P3, U6.R1IN
- net SCK: now also JP2.6; no longer IC1.CLK, JP1.6
- net SCL: now also HT16K1.SCL, IC1.SCL, JP4.11, R40.2; no longer IC2.SCL, JP3.11
- net SDA: now also HT16K1.SDA, IC1.SDA, JP4.12, R41.2; no longer IC2.SDA, JP3.12
- net TXD: now also DE9FEMALE1.P4, U1.T1OUT; no longer DE9FEMALE.P4, U6.T1OUT
- net UART_RX: now also JP2.3, U1.R1OUT; no longer JP1.3, U6.R1OUT
- net UART_TX: now also JP2.2, U1.T1IN; no longer JP1.2, U6.T1IN
- net VBAT: now also JP4.1; no longer JP3.1
- net VBUS: now also JP4.3; no longer JP3.3
Other:
- note removed: "Standoffs!"
- moved on the sheet: C1, C2, C3
